File: NCD57201DR2G_breakout/NCD57201DR2G_breakout.kicad_pcb (KiCad board)
At the start: 2 copper layers, 17.8 x 15.2 mm, 4 parts, among them IC1 NCD57201DR2G, J1 Conn_01x04, J2 Conn_01x04

Commit message: Some updates.
Routing:
- net /LIN: track 5.19 -> 0.00 mm
- net /HIN: track 5.16 -> 0.00 mm
Changed lines of the file:
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@@
   (segment (start 113.3406 68.7324) (end 110.3022 68.7324) (width 0.3) (layer "F.Cu") (net 1))
   (segment (start 110.3022 68.7324) (end 108.4326 66.8628) (width 0.3) (layer "F.Cu") (net 1))
-  (segment (start 109.0322 70.0024) (end 108.4326 69.4028) (width 0.2) (layer "F.Cu") (net 3))
-  (segment (start 113.3406 70.0024) (end 109.0322 70.0024) (width 0.2) (layer "F.Cu") (net 3))
-  (segment (start 108.4326 71.9428) (end 109.103 71.2724) (width 0.2) (layer "F.Cu") (net 4))
-  (segment (start 109.103 71.2724) (end 113.3406 71.2724) (width 0.2) (layer "F.Cu") (net 4))
   (segment (start 121.7322 72.5424) (end 123.6726 74.4828) (width 0.8) (layer "F.Cu") (net 5))
   (segment (start 118.7646 72.5424) (end 121.7322 72.5424) (width 0.8) (layer "F.Cu") (net 5))

Commit message: Pretty much done.
Parts:
- IC1: footprint antesc:SOIC127P600X175-8N -> breakouts:SOIC127P600X175-8N
- REF**: value OSHW-Logo2_14.6x12mm_SilkScreen -> OSHW-Logo2_7.3x6mm_SilkScreen; footprint Symbol:OSHW-Logo2_14.6x12mm_SilkScreen -> Symbol:OSHW-Logo2_7.3x6mm_SilkScreen
- moved REF** 2.85 mm to (116.1, 75.0)
Connections:
- net GND renamed GND1
Routing:
- net GND1: track 0.00 -> 5.71 mm, vias 0 -> 1
- net /LIN: track 0.00 -> 5.19 mm
- net /HIN: track 0.00 -> 5.16 mm
- added copper zone on B.Cu, net GND1
- removed copper zone on B.Cu, net +5V
