File: NCD57201DR2G_breakout/NCD57201DR2G_breakout.kicad_sch (KiCad schematic)
At the start: 3 parts, among them IC1 NCD57201DR2G, J1 Conn_01x04, J2 Conn_01x04

Commit message: Some updates.
Other:
- moved on the sheet: J1
Changed lines of the file:
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@@
     (stroke (width 0) (type default))
   )
-  (wire (pts (xy 63.5 53.34) (xy 66.04 53.34))
-    (stroke (width 0) (type default))
-  )
-  (wire (pts (xy 63.5 50.8) (xy 64.77 50.8))
-    (stroke (width 0) (type default))
-  )
-  (wire (pts (xy 63.5 55.88) (xy 66.04 55.88))
-    (stroke (width 0) (type default))
-  )
-  (wire (pts (xy 63.5 58.42) (xy 64.77 58.42))
+  (wire (pts (xy 38.1 53.34) (xy 66.04 53.34))
+    (stroke (width 0) (type default))
+  )
+  (wire (pts (xy 38.1 55.88) (xy 66.04 55.88))
+    (stroke (width 0) (type default))
+  )
+  (wire (pts (xy 38.1 50.8) (xy 64.77 50.8))
     (stroke (width 0) (type default))
   )
@@
     (stroke (width 0) (type default))
   )
+  (wire (pts (xy 38.1 58.42) (xy 64.77 58.42))
+    (stroke (width 0) (type default))
+  )
   (label "LIN" (at 64.262 55.88 0) (fields_autoplaced)
     (effects (font (size 1.27 1.27)) (justify left bottom))
@@
       (effects (font (size 1.27 1.27)) hide)
     )
-    (property "Value" "PWR_FLAG" (at 51.562 38.1 0)
-      (effects (font (size 1.27 1.27)))
+    (property "Value" "PWR_FLAG" (at 53.34 34.29 0)
+      (effects (font (size 1.27 1.27)) (justify right))
     )
     (property "Footprint" "" (at 51.562 33.02 0)
@@
       (effects (font (size 1.27 1.27)) hide)
     )
-    (property "Value" "GND" (at 44.45 38.1 0)
-      (effects (font (size 1.27 1.27)))
+    (property "Value" "GND" (at 46.99 34.29 0)
+      (effects (font (size 1.27 1.27)) (justify left))
     )
     (property "Footprint" "" (at 44.45 33.02 0)
@@
     )
   )
-  (symbol (lib_id "Connector_Generic:Conn_01x04") (at 58.42 53.34 0) (mirror y) (unit 1)
-    (in_bom yes) (on_board yes) (dnp no)
-    (property "Reference" "J1" (at 56.388 53.34 0)
-      (effects (font (size 1.27 1.27)) (justify left))
-    )
-    (property "Value" "Conn_01x04" (at 56.388 55.88 0)
-      (effects (font (size 1.27 1.27)) (justify left))
-    )
-    (property "Footprint" "Connector_PinHeader_2.54mm:PinHeader_1x04_P2.54mm_Vertical" (at 58.42 53.34 0)
-      (effects (font (size 1.27 1.27)) hide)
-    )
-    (property "Datasheet" "~" (at 58.42 53.34 0)
+  (symbol (lib_id "Connector_Generic:Conn_01x04") (at 33.02 53.34 0) (mirror y) (unit 1)
+    (in_bom yes) (on_board yes) (dnp no) (fields_autoplaced)
+    (property "Reference" "J1" (at 33.02 44.45 0)
+      (effects (font (size 1.27 1.27)))
+    )
+    (property "Value" "Conn_01x04" (at 33.02 46.99 0)
+      (effects (font (size 1.27 1.27)))
+    )
+    (property "Footprint" "Connector_PinHeader_2.54mm:PinHeader_1x04_P2.54mm_Vertical" (at 33.02 53.34 0)
+      (effects (font (size 1.27 1.27)) hide)
+    )
+    (property "Datasheet" "~" (at 33.02 53.34 0)
       (effects (font (size 1.27 1.27)) hide)
     )
@@
       (effects (font (size 1.27 1.27)) hide)
     )
-    (property "Value" "-BATT" (at 92.71 66.04 0)
-      (effects (font (size 1.27 1.27)))
+    (property "Value" "-BATT" (at 95.25 62.23 0)
+      (effects (font (size 1.27 1.27)) (justify right))
     )
     (property "Footprint" "" (at 92.71 60.96 0)
@@
   (symbol (lib_id "Connector_Generic:Conn_01x04") (at 99.06 53.34 0) (unit 1)
     (in_bom yes) (on_board yes) (dnp no) (fields_autoplaced)
-    (property "Reference" "J2" (at 101.854 53.34 0)
-      (effects (font (size 1.27 1.27)) (justify left))
-    )
-    (property "Value" "Conn_01x04" (at 101.854 55.88 0)
+    (property "Reference" "J2" (at 101.6 53.34 0)
+      (effects (font (size 1.27 1.27)) (justify left))
+    )
+    (property "Value" "Conn_01x04" (at 101.6 55.88 0)
       (effects (font (size 1.27 1.27)) (justify left))
     )
@@
       (effects (font (size 1.27 1.27)) hide)
     )
-    (property "Value" "+BATT" (at 91.44 43.18 0)
-      (effects (font (size 1.27 1.27)))
+    (property "Value" "+BATT" (at 93.98 46.99 0)
+      (effects (font (size 1.27 1.27)) (justify left))
     )
     (property "Footprint" "" (at 91.44 48.26 0)
@@
       (effects (font (size 1.27 1.27)) hide)
     )
-    (property "Value" "+5V" (at 51.562 27.94 0)
-      (effects (font (size 1.27 1.27)))
+    (property "Value" "+5V" (at 53.34 31.75 0)
+      (effects (font (size 1.27 1.27)) (justify left))
     )
     (property "Footprint" "" (at 51.562 33.02 0)

Commit message: Pretty much done.
Parts:
- added C1: 100n, symbol Device:C
- added C2: 10u, symbol Device:C
- added TP1: TestPoint, TestPoint:TestPoint_Pad_D1.0mm, symbol Connector:TestPoint
Connections:
- net +5V: now also C1.1, C2.1
- net GND: no longer IC1.4 (GND), J1.4 (Pin_4)
- new net GND1: C1.2, C2.2, IC1.4 (GND), J1.4 (Pin_4), TP1.1
Other:
- moved on the sheet: IC1, J1, J2
